File: KapiBara3_mainBoard.kicad_sch (KiCad schematic)
At the start: 0 parts

Commit message: I need to think what else to add
Parts:
- added TP14, TP15, TP16, TP17: TestPoint, TestPoint:TestPoint_Pad_D3.0mm, symbol Connector:TestPoint
Connections:
- new net GND: TP14.1, TP15.1, TP16.1, TP17.1
