File: connector.kicad_sch (KiCad schematic)
At the start: 8 parts, among them J1 Conn_02x20_Top_Bottom, J2 Conn_02x20_Top_Bottom, J3 Conn_02x20_Top_Bottom, J4 Conn_02x20_Top_Bottom, J6 Conn_01x02, J7 Conn_01x08, J8 Conn_01x02, J9 Conn_01x02

Commit message: I need to think what else to add
Parts:
- added D10, D11, D12, D13, D14, D15, D4, D5, D6, D7, D8, D9: TVS, Diode_SMD:D_SOD-323, symbol Device:D
- added TP1, TP10, TP11, TP2, TP4, TP5, TP6, TP7, TP8, TP9: TestPoint, TestPoint:TestPoint_Pad_D1.5mm, symbol Connector:TestPoint
Connections:
- net D1+: now also D5.1 (K), TP2.1
- net D1-: now also D4.1 (K), TP1.1
- net D2+: now also D7.1 (K), TP4.1
- net D2-: now also D6.1 (K), TP5.1
- net D3+: now also D9.1 (K), TP6.1
- net D3-: now also D8.1 (K), TP7.1
- net D4+: now also D11.1 (K), TP8.1
- net D4-: now also D10.1 (K), TP9.1
- net D_1+: now also D12.1 (K), TP10.1
- net D_1-: now also D13.1 (K), TP11.1
- net GND: now also D10.2 (A), D11.2 (A), D12.2 (A), D13.2 (A), D14.2 (A), D15.2 (A), D4.2 (A), D5.2 (A), D6.2 (A), D7.2 (A), D8.2 (A), D9.2 (A)
- new net D_2+: D14.1 (K)
- new net D_2-: D15.1 (K)

Commit message: I have shrinken down the board
Parts:
- removed J1, J2, J3, J4: Conn_02x20_Top_Bottom, Connector_IDC:IDC-Header_2x20_P2.54mm_Vertical, symbol Connector_Generic:Conn_02x20_Top_Bottom
- added J1, J2, J3, J4: Conn_01x04_MountingPin, Connector_FFC-FPC:Amphenol_F32Q-1A7x1-11004_1x04-1MP_P0.5mm_Horizontal, symbol Connector_Generic_MountingPin:Conn_01x04_MountingPin
- added J10, J11, J12, J13, J14: Conn_01x02, Connector_AMASS:AMASS_XT30U-F_1x02_P5.0mm_Vertical, symbol Connector_Generic:Conn_01x02
- J6: footprint Connector_AMASS:AMASS_XT60PW-F_1x02_P7.20mm_Horizontal -> Connector_AMASS:AMASS_XT60-M_1x02_P7.20mm_Vertical
Connections:
- net D1+: now also J3.3 (Pin_3)
- net D1-: now also J3.2 (Pin_2)
- net D2+: now also J2.3 (Pin_3)
- net D2-: now also J2.2 (Pin_2)
- net D3+: now also J1.3 (Pin_3)
- net D3-: now also J1.2 (Pin_2)
- net D4+: now also J4.3 (Pin_3)
- net D4-: now also J4.2 (Pin_2)
- net GND: now also J1.1 (Pin_1), J1.4 (Pin_4), J1.MP (MountPin), J10.1 (Pin_1), J11.1 (Pin_1), J12.1 (Pin_1), J13.1 (Pin_1), J14.1 (Pin_1), J2.1 (Pin_1), J2.4 (Pin_4), J2.MP (MountPin), J3.1 (Pin_1), J3.4 (Pin_4), J3.MP (MountPin), J4.1 (Pin_1), J4.4 (Pin_4), J4.MP (MountPin)
- net VCC: now also J10.2 (Pin_2), J11.2 (Pin_2), J12.2 (Pin_2), J13.2 (Pin_2), J14.2 (Pin_2)
Other:
- note added: "Main Power Connector"
- moved on the sheet: J6, J7
