File: power_switch.kicad_sch (KiCad schematic)
At the start: 8 parts, among them Q1 Q_PMOS_GDS, Q2 2N7002, Q3 Q_PMOS_GDS

Commit message: I need to think what else to add
Parts:
- added D2, D3: LED, LED_SMD:LED_0805_2012Metric_Pad1.15x1.40mm_HandSolder, symbol Device:LED
- added R11, R12: 1k, Resistor_SMD:R_0603_1608Metric, symbol Device:R
- added TP13: TestPoint, TestPoint:TestPoint_Pad_1.5x1.5mm, symbol Connector:TestPoint
Connections:
- net GND: now also D2.1 (K), D3.1 (K)
- net VCC: now also R12.1
- net VDD: now also R11.1, TP13.1
- new net: D3.2 (A), R12.2
- new net: D2.2 (A), R11.2
