File: usb_hub.kicad_sch (KiCad schematic)
At the start: 20 parts, among them U1 SL2.1A, U2 AP63300WU-7, Y1 12Mhz

Commit message: I need to think what else to add
Parts:
- added C12, C13, C14: 22u, Capacitor_SMD:C_0805_2012Metric_Pad1.18x1.45mm_HandSolder, symbol Device:C
- added TP12: TestPoint, TestPoint:TestPoint_Pad_1.5x1.5mm, symbol Connector:TestPoint
Connections:
- net GND: now also C12.2, C13.2, C14.2
- net VCC: now also C12.1, C13.1, C14.1, TP12.1

Commit message: Final design
Parts:
- R1: value 52.5k -> 300k
- R2: value 10k -> 56k
Changed lines of the file:
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@@
 			)
 		)
-		(property "Value" "52.5k"
+		(property "Value" "300k"
 			(at 139.065 49.5299 0)
 			(effects
@@
 			)
 		)
-		(property "Value" "10k"
+		(property "Value" "56k"
 			(at 139.065 59.6899 0)
 			(effects
